Commit message: Trayectorias segundo corte, Trayectorias con el robot físico Y README del proyecto

File: RobotUtadeo/urdf/xacro/lesson_urdf/urdf/Robot_Utadeo.urdf (robot description, URDF)
Before this commit: robot My_Robot, 7 links, 6 joints
Joints:
- joint joint_1: limit lower=0 upper=62.8319 effort=5.0 velocity=5.0 -> lower=-1.57 upper=1.57 effort=5.0 velocity=5.0
