Commit message: Update BrazoRobotico.urdf

File: BrazoRobotico/urdf/xacro/lesson_urdf/urdf/BrazoRobotico.urdf (robot description, URDF)
Before this commit: robot My_Robot, 7 links, 6 joints
Links:
- link Gripper: geometry visual mesh filename=package://lesson_urdf/meshes/visual/gripper.stl scale=0.1 0.1 0.1
- link link_4: geometry visual mesh filename=package://lesson_urdf/meshes/visual/Muneca.stl scale=0.1 0.1 0.1
